File: jensx1000.kicad_pcb (KiCad board)
At the start: 2 copper layers, 101 x 38.8 mm, 305 parts, among them J1 Conn_01x03_Pin, J2 Conn_01x04_Pin, J3 Conn_01x12_Pin, J5 Conn_01x09_Pin, J6 Conn_01x11_Pin, J7 Conn_01x11_Pin, J8 Conn_01x06_Pin, J9 Conn_01x07_Pin, Q1 BC309C, Q2 BC237, Q3 BC237, Q4 BC307, Q5 PN2222A, Q6 BC309, Q7 BC309, Q8 BC239, SW1 SW_SP3T, SW10 SW_SPST, SW11 SW_SPST, SW12 SW_SPST, SW13 SW_SPST, SW14 SW_SPST, SW15 SW_SPST, SW16 SW_SPST, SW17 SW_SPST, SW18 SW_SPST, SW19 SW_SPST, SW2 SW_Rotary_1x3_MP, SW20 SW_SPST, SW21 SW_SPST, SW22 SW_SPST, SW23 SW_SPST, SW24 SW_SPST, SW25 SW_SPST, SW26 SW_SPST, SW27 SW_SPST, SW28 SW_SPST, SW29 SW_SPST, SW3 SW_SPST, SW30 SW_SPST, SW31 SW_SPST, SW32 SW_SPST, SW33 SW_SPST, SW34 SW_SPST, SW35 SW_SPST, SW36 SW_SPST, SW37 SW_SPST, SW38 SW_SPST, SW39 SW_SPST, SW4 SW_SPST, SW40 2P4T, SW5 SW_SPST, SW6 SW_SPST, SW7 SW_SPST, SW8 SW_SPST, SW9 SW_SPST, U1 L7912, U10 4013, U11 4001, U12 4066, U13 Opamp_Dual, U14 74LS221, U15 4066, U16 LF353, U17 M110, U19 Opamp_Dual, U2 L7812, U20 LF351N, U21 LM301, U22 LM301, U24 LM13700, U25 LM13700, U26 LM741, U3 L7805, U4 Opamp_Dual, U5 MM5837, U6 CA3080, U7 LM741, U8 4001, U9 Opamp_Dual

Commit message: Move components around
Parts:
- moved R18 187.4 mm to (370.1, -141.2)
- moved R19 187.4 mm to (370.1, -138.1)
- moved R21 187.4 mm to (370.1, -131.8)
- moved R23 187.4 mm to (370.1, -125.5)
- moved R24 187.4 mm to (370.1, -122.3)
- moved R20 187.4 mm to (370.1, -134.9)
- moved R22 187.4 mm to (370.1, -128.6)
- moved R62 178.2 mm to (214.9, -151.5), turned to 180 degrees
- moved R61 177.0 mm to (212.6, -158.2)
- moved J6 157.7 mm to (192.0, -163.4)
- moved U8 149.1 mm to (228.5, -144.5)
- moved D5 147.4 mm to (380.1, -153.2)
- moved C16 147.4 mm to (389.8, -149.4)
- moved CP15 147.4 mm to (381.6, -146.7)
- moved CP19 145.9 mm to (198.5, -152.8)
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
Commit message: Move components around
Parts:
- moved U16 467.0 mm to (251.4, 62.6), turned to 180 degrees
- moved D11 422.8 mm to (51.9, 290.6), turned to 90 degrees
- moved D12 418.1 mm to (55.8, 290.6), turned to 90 degrees
- moved C36 416.6 mm to (200.8, 70.5)
- moved C35 416.5 mm to (200.8, 64.0)
- moved C33 416.3 mm to (200.5, 57.5)
- moved C32 416.2 mm to (200.5, 50.8)
- moved C31 416.0 mm to (200.5, 44.0)
- moved C30 415.7 mm to (200.2, 37.2)
- moved D13 413.3 mm to (59.8, 290.6), turned to 90 degrees
- moved C37 409.9 mm to (188.5, 121.4)
- moved D14 408.6 mm to (63.7, 290.6), turned to 90 degrees
- moved J7 406.7 mm to (200.5, 28.6), turned to -90 degrees
- moved SW3 405.1 mm to (51.8, 278.3), turned to 90 degrees
- moved D15 403.9 mm to (67.6, 290.6), turned to 90 degrees
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Other:
- board text added: "ATTACK"
- board text added: "DECAY"
- board text added: "ENV. LEVEL"
- board text added: "GLIDE"
- board text added: "LEVEL"
- board text added: "LFO"
- board text added: "LFO SPEED"
- board text added: "NOISE"
- board text added: "OCTAVE"
- board text added: "PULSE WIDTH"
- board text added: "PWM"
- board text added: "RELEASE"
- board text added: "RESONANCE"
- board text added: "SUSTAIN"
- board text added: "TUNE"
- board text added: "VIBRATO"
- board text added: "VOLUME"
- board text added: "WAVEFORM"

Commit message: Move components around
Parts:
- moved J3 353.0 mm to (521.3, 309.3), turned to -90 degrees
- moved R74 332.2 mm to (503.2, 275.4), turned to 90 degrees
- moved D47 328.2 mm to (519.4, 259.2)
- moved SW39 328.1 mm to (519.4, 246.8)
- moved R73 327.8 mm to (499.1, 275.4), turned to 90 degrees
- moved R106 327.2 mm to (496.7, 267.7), turned to -90 degrees
- moved R107 325.2 mm to (494.3, 267.7), turned to -90 degrees
- moved R108 323.1 mm to (491.7, 267.7), turned to -90 degrees
- moved R109 321.0 mm to (489.1, 267.7), turned to -90 degrees
- moved D46 320.5 mm to (507.7, 259.2)
- moved SW38 320.4 mm to (507.7, 246.9)
- moved D45 312.7 mm to (496.1, 259.2)
- moved SW37 312.7 mm to (496.1, 246.9)
- moved D44 305.0 mm to (484.4, 259.2)
- moved SW36 305.0 mm to (484.4, 246.9)
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