File: vco.kicad_sch (KiCad schematic)
At the start: 72 parts, among them J4 Conn_01x09_Pin, J7 Conn_01x11_Pin, Q5 PN2222A, Q6 BC309, Q7 BC309, Q8 BC239, SW2 SW_Rotary_1x3_MP, SW40 2P4T, U10 4013, U14 74LS221, U16 LF353, U21 LM301, U22 LM301, U26 LM741

Commit message: Routing
Parts:
- R69, R77, R80, R83, R88, R90, R91, R92: footprint Resistor_THT:R_Axial_DIN0207_L6.3mm_D2.5mm_P15.24mm_Horizontal -> Resistor_THT:R_Axial_DIN0309_L9.0mm_D3.2mm_P12.70mm_Horizontal
Changed lines of the file:
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@@
 			)
 		)
-		(property "Footprint" "Resistor_THT:R_Axial_DIN0207_L6.3mm_D2.5mm_P15.24mm_Horizontal"
+		(property "Footprint" "Resistor_THT:R_Axial_DIN0309_L9.0mm_D3.2mm_P12.70mm_Horizontal"
 			(at 325.12 201.422 90)
 			(effects
@@
 			)
 		)
-		(property "Footprint" "Resistor_THT:R_Axial_DIN0207_L6.3mm_D2.5mm_P15.24mm_Horizontal"
+		(property "Footprint" "Resistor_THT:R_Axial_DIN0309_L9.0mm_D3.2mm_P12.70mm_Horizontal"
 			(at 287.782 172.72 90)
 			(effects
@@
 			)
 		)
-		(property "Footprint" "Resistor_THT:R_Axial_DIN0207_L6.3mm_D2.5mm_P15.24mm_Horizontal"
+		(property "Footprint" "Resistor_THT:R_Axial_DIN0309_L9.0mm_D3.2mm_P12.70mm_Horizontal"
 			(at 146.05 99.568 90)
 			(effects
@@
 			)
 		)
-		(property "Footprint" "Resistor_THT:R_Axial_DIN0207_L6.3mm_D2.5mm_P15.24mm_Horizontal"
+		(property "Footprint" "Resistor_THT:R_Axial_DIN0309_L9.0mm_D3.2mm_P12.70mm_Horizontal"
 			(at 173.228 184.15 90)
 			(effects
@@
 			)
 		)
-		(property "Footprint" "Resistor_THT:R_Axial_DIN0207_L6.3mm_D2.5mm_P15.24mm_Horizontal"
+		(property "Footprint" "Resistor_THT:R_Axial_DIN0309_L9.0mm_D3.2mm_P12.70mm_Horizontal"
 			(at 207.01 180.848 90)
 			(effects
@@
 			)
 		)
-		(property "Footprint" "Resistor_THT:R_Axial_DIN0207_L6.3mm_D2.5mm_P15.24mm_Horizontal"
+		(property "Footprint" "Resistor_THT:R_Axial_DIN0309_L9.0mm_D3.2mm_P12.70mm_Horizontal"
 			(at 223.52 177.292 90)
 			(effects
@@
 			)
 		)
-		(property "Footprint" "Resistor_THT:R_Axial_DIN0207_L6.3mm_D2.5mm_P15.24mm_Horizontal"
+		(property "Footprint" "Resistor_THT:R_Axial_DIN0309_L9.0mm_D3.2mm_P12.70mm_Horizontal"
 			(at 227.33 89.408 90)
 			(effects
@@
 			)
 		)
-		(property "Footprint" "Resistor_THT:R_Axial_DIN0207_L6.3mm_D2.5mm_P15.24mm_Horizontal"
+		(property "Footprint" "Resistor_THT:R_Axial_DIN0309_L9.0mm_D3.2mm_P12.70mm_Horizontal"
 			(at 358.14 202.438 90)
 			(effects

Commit message: Routing
Parts:
- R67, R68: footprint Resistor_THT:R_Axial_DIN0207_L6.3mm_D2.5mm_P15.24mm_Horizontal -> Resistor_THT:R_Axial_DIN0309_L9.0mm_D3.2mm_P12.70mm_Horizontal
Connections:
- net +12V: now also RT27.3, U10.14 (VDD); no longer RT27.1
- net +5V: now also RT21.3; no longer RT21.1, U10.14 (VDD)
- net -12V: now also RT27.1; no longer RT27.3
- net GND: now also RT21.1; no longer RT21.3
- net at R99.2, U22.2 (-): now also RT28.3; no longer RT28.1
Other:
- moved on the sheet: RT21, RT28
Changed lines of the file:
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@@
 	)
 	(junction
-		(at 54.61 26.67)
+		(at 284.48 124.46)
 		(diameter 0)
 		(color 0 0 0 0)
 	)
 	(junction
-		(at 284.48 124.46)
+		(at 252.73 167.64)
 		(diameter 0)
 		(color 0 0 0 0)
 	)
 	(junction
-		(at 252.73 167.64)
+		(at 87.63 27.94)
 		(diameter 0)
 		(color 0 0 0 0)
@@
 	(wire
 		(pts
-			(xy 54.61 25.4) (xy 54.61 26.67)
+			(xy 54.61 25.4) (xy 54.61 27.94)
 		)
 		(stroke
@@
 	(wire
 		(pts
+			(xy 73.66 30.48) (xy 73.66 27.94)
+		)
+		(stroke
+			(width 0)
+			(type default)
+		)
+	)
+	(wire
+		(pts
 			(xy 393.7 200.66) (xy 386.08 200.66)
 		)
@@
 	(wire
 		(pts
-			(xy 87.63 26.67) (xy 87.63 33.02)
+			(xy 87.63 26.67) (xy 87.63 27.94)
 		)
 		(stroke
@@
 	(wire
 		(pts
+			(xy 73.66 27.94) (xy 87.63 27.94)
+		)
+		(stroke
+			(width 0)
+			(type default)
+		)
+	)
+	(wire
+		(pts
 			(xy 156.21 130.81) (xy 163.83 130.81)
 		)
@@
 	(wire
 		(pts
+			(xy 87.63 27.94) (xy 87.63 33.02)
+		)
+		(stroke
+			(width 0)
+			(type default)
+		)
+	)
+	(wire
+		(pts
 			(xy 275.59 167.64) (xy 278.13 167.64)
 		)
@@
 	(wire
 		(pts
-			(xy 54.61 26.67) (xy 73.66 26.67)
-		)
-		(stroke
-			(width 0)
-			(type default)
-		)
-	)
-	(wire
-		(pts
 			(xy 156.21 130.81) (xy 156.21 132.08)
 		)
@@
 	(wire
 		(pts
-			(xy 73.66 30.48) (xy 73.66 26.67)
-		)
-		(stroke
-			(width 0)
-			(type default)
-		)
-	)
-	(wire
-		(pts
 			(xy 24.13 177.8) (xy 30.48 177.8)
 		)
@@
 	(wire
 		(pts
-			(xy 54.61 26.67) (xy 54.61 27.94)
-		)
-		(stroke
-			(width 0)
-			(type default)
-		)
-	)
-	(wire
-		(pts
 			(xy 127 180.34) (xy 127 186.69)
 		)
@@
 		)
 	)
+	(label "LFO_OUT"
+		(at 24.13 213.36 180)
+		(fields_autoplaced yes)
+		(effects
+			(font
+				(size 1.27 1.27)
+			)
+			(justify right bottom)
+		)
+		(property "Netclass" "LFO_OUT"
+			(at 24.13 214.63 0)
+			(effects
+				(font
+					(size 1.27 1.27)
+					(italic yes)
+				)
+				(justify right)
+			)
+		)
+	)
 	(label "DC"
 		(at 26.67 49.53 0)
@@
 		)
 	)
-	(hierarchical_label "LFO_OUT"
-		(shape output)
-		(at 24.13 213.36 180)
-		(effects
-			(font
-				(size 1.27 1.27)
-			)
-			(justify right)
-		)
-	)
 	(hierarchical_label "GND"
 		(shape input)
@@
 			)
 		)
-		(property "Footprint" "Resistor_THT:R_Axial_DIN0207_L6.3mm_D2.5mm_P15.24mm_Horizontal"
+		(property "Footprint" "Resistor_THT:R_Axial_DIN0309_L9.0mm_D3.2mm_P12.70mm_Horizontal"
 			(at 45.72 102.108 90)
 			(effects
@@
 		(lib_id "Device:R_Potentiometer_Trim")
 		(at 266.7 124.46 0)
+		(mirror x)
 		(unit 1)
 		(exclude_from_sim no)
@@
 		(dnp no)
 		(property "Reference" "RT27"
-			(at 264.16 123.1899 0)
+			(at 264.16 125.7301 0)
 			(effects
 				(font
@@
 		)
 		(property "Value" "10K"
-			(at 264.16 125.7299 0)
+			(at 264.16 123.1901 0)
 			(effects
 				(font
@@
 	(symbol
 		(lib_id "Device:R_Potentiometer_Trim")
-		(at 299.72 124.46 90)
+		(at 299.72 124.46 270)
+		(mirror x)
 		(unit 1)
 		(exclude_from_sim no)
@@
 		(on_board yes)
 		(dnp no)
-		(fields_autoplaced yes)
 		(property "Reference" "RT28"
 			(at 299.72 128.27 90)
@@
 			)
 		)
-		(property "Footprint" "Resistor_THT:R_Axial_DIN0207_L6.3mm_D2.5mm_P15.24mm_Horizontal"
+		(property "Footprint" "Resistor_THT:R_Axial_DIN0309_L9.0mm_D3.2mm_P12.70mm_Horizontal"
 			(at 35.56 102.108 90)
 			(effects
@@
 	(symbol
 		(lib_id "Device:R_Potentiometer_Trim")
-		(at 59.69 100.33 0)
-		(mirror y)
+		(at 59.69 100.33 180)
 		(unit 1)
 		(exclude_from_sim no)
@@
 		(dnp no)
 		(property "Reference" "RT21"
-			(at 62.23 99.0599 0)
+			(at 62.23 101.6001 0)
 			(effects
 				(font
@@
 		)
 		(property "Value" "10K"
-			(at 62.23 101.5999 0)
+			(at 62.23 99.0601 0)
 			(effects
 				(font
