File: vco.kicad_sch (KiCad schematic)
At the start: 72 parts, among them J4 Conn_01x09_Pin, J7 Conn_01x11_Pin, Q5 PN2222A, Q6 BC309, Q7 BC309, Q8 BC239, SW2 SW_Rotary_1x3_MP, SW40 2P4T, U10 4013, U14 74LS221, U16 LF353, U21 LM301, U22 LM301, U26 LM741

Commit message: Fix VCF layout, routing, adding pads for switches
Parts:
- added C4, C5: 10uF, Capacitor_THT:CP_Radial_D8.0mm_P3.80mm, symbol Device:C_Polarized
- added H10, H11, H12, H13, H14, H15, H16, H4, H5, H6, H7, H8, H9: MountingHole_Pad, MountingHole:MountingHole_2.2mm_M2_Pad, symbol Mechanical:MountingHole_Pad
Connections:
- net +12V: now also C4.1
- net -12V: now also C5.2
- net 16': now also H15.1
- net 2': now also H12.1
- net 4': now also H13.1
- net 8': now also H14.1
- net GND: now also C4.2, C5.1, H11.1
- net PULSE: now also H9.1
- net SAW: now also H8.1
- net SQR: now also H7.1
- net at C30.1, R76.2, SW40.1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: now also H16.1
- net at R95.1, SW40.9: now also H4.1
- net at R94.1, SW40.8: now also H5.1
- net at RV24.3, SW2.4: now also H10.1
- net at R92.1, SW40.7: now also H6.1

Commit message: Fixed VCF TRIG/GATE net, routed all except keyboard
Parts:
- R110: footprint Resistor_THT:R_Axial_DIN0207_L6.3mm_D2.5mm_P15.24mm_Horizontal -> Resistor_THT:R_Axial_DIN0207_L6.3mm_D2.5mm_P10.16mm_Horizontal
Connections:
- net LFO_OUT is gone; now on net FROM_LFO: J4.4 (Pin_4)
Changed lines of the file:
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@@
 	(wire
 		(pts
+			(xy 24.13 73.66) (xy 27.94 73.66)
+		)
+		(stroke
+			(width 0)
+			(type default)
+		)
+	)
+	(wire
+		(pts
 			(xy 101.6 191.77) (xy 101.6 208.28)
 		)
@@
 	(wire
 		(pts
+			(xy 24.13 213.36) (xy 30.48 213.36)
+		)
+		(stroke
+			(width 0)
+			(type default)
+		)
+	)
+	(wire
+		(pts
 			(xy 149.86 97.79) (xy 152.4 97.79)
 		)
@@
 	(wire
 		(pts
-			(xy 24.13 213.36) (xy 30.48 213.36)
-		)
-		(stroke
-			(width 0)
-			(type default)
-		)
-	)
-	(wire
-		(pts
 			(xy 25.4 245.11) (xy 25.4 247.65)
 		)
@@
 		)
 	)
+	(label "LFO_OUT"
+		(at 27.94 73.66 0)
+		(effects
+			(font
+				(size 1.27 1.27)
+			)
+			(justify left bottom)
+		)
+	)
 	(label "16'"
 		(at 92.71 208.28 0)
@@
 	(label "LFO_OUT"
 		(at 24.13 213.36 180)
-		(fields_autoplaced yes)
 		(effects
 			(font
@@
 			(justify right bottom)
 		)
-		(property "Netclass" "LFO_OUT"
-			(at 24.13 214.63 0)
-			(effects
-				(font
-					(size 1.27 1.27)
-					(italic yes)
-				)
-				(justify right)
-			)
-		)
 	)
 	(label "DC"
@@
 		)
 	)
+	(label "LFO_OUT"
+		(at 375.92 132.08 0)
+		(effects
+			(font
+				(size 1.27 1.27)
+			)
+			(justify left bottom)
+		)
+	)
 	(label "GND"
 		(at 157.48 195.58 180)
@@
 		)
 	)
+	(label "LFO_OUT"
+		(at 156.21 91.44 0)
+		(effects
+			(font
+				(size 1.27 1.27)
+			)
+			(justify left bottom)
+		)
+	)
 	(label "PULSE"
 		(at 354.33 72.39 180)
@@
 	(hierarchical_label "FROM_LFO"
 		(shape input)
-		(at 156.21 91.44 0)
+		(at 24.13 73.66 180)
 		(effects
 			(font
 				(size 1.27 1.27)
 			)
-			(justify left)
+			(justify right)
 		)
 	)
@@
 		)
 	)
-	(hierarchical_label "FROM_LFO"
-		(shape input)
-		(at 375.92 132.08 0)
-		(effects
-			(font
-				(size 1.27 1.27)
-			)
-			(justify left)
-		)
-	)
 	(hierarchical_label "GND"
 		(shape input)
@@
 			)
 		)
-		(property "Footprint" "Resistor_THT:R_Axial_DIN0207_L6.3mm_D2.5mm_P15.24mm_Horizontal"
+		(property "Footprint" "Resistor_THT:R_Axial_DIN0207_L6.3mm_D2.5mm_P10.16mm_Horizontal"
 			(at 387.35 80.772 90)
 			(effects
