File: vco.kicad_sch (KiCad schematic)
At the start: 87 parts, among them J4 Conn_01x09_Pin, J7 Conn_01x11_Pin, Q5 PN2222A, Q6 BC309, Q7 BC309, Q8 BC239, SW2 SW_Rotary_1x3_MP, SW40 2P4T, U10 4013, U14 74LS221, U16 LF353, U21 LM301, U22 LM301, U26 LM741

Commit message: Update README, add license to sheets
Other:
- note added: "NOTE: Not R110 on schematic, but present on board"
- note added: "NOTE: Not on schematic, but present on board"
- note added: "R76 and C30 are not present on PCB"
- note removed: "NOTE: Not on schematic"
- title: (none) -> JEN SX-1000
Changed lines of the file:
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@@
 	(generator_version "9.0")
 	(paper "A3")
+	(title_block
+		(title "JEN SX-1000")
+		(comment 1 "SPDX-License-Identifier: CERN-OHL-S-2.0")
+	)
 	(rectangle
 		(start 15.24 82.55)
@@
 			(type color)
 			(color 255 255 194 1)
+		)
+	)
+	(rectangle
+		(start 124.46 184.15)
+		(end 146.05 201.93)
+		(stroke
+			(width 0)
+			(type default)
+		)
+		(fill
+			(type none)
 		)
 	)
@@
 		)
 	)
-	(text "NOTE: Not on schematic"
+	(text "NOTE: Not on schematic, but\npresent on board"
 		(exclude_from_sim no)
-		(at 58.166 250.952 0)
+		(at 57.658 241.3 0)
 		(effects
 			(font
@@
 		(exclude_from_sim no)
 		(at 382.778 113.538 0)
+		(effects
+			(font
+				(size 1.27 1.27)
+			)
+		)
+	)
+	(text "R76 and C30 are not present on PCB"
+		(exclude_from_sim no)
+		(at 148.336 179.07 0)
 		(effects
 			(font
@@
 		)
 	)
-	(text "NOTE: Not on schematic"
+	(text "NOTE: Not R110 on schematic, \nbut present on board"
 		(exclude_from_sim no)
-		(at 401.828 78.232 0)
+		(at 392.938 88.138 0)
 		(effects
 			(font

Commit message: Update sheets
Other:
- company: (none) -> Csaba Nagy
Changed lines of the file:
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@@
 	(title_block
 		(title "JEN SX-1000")
+		(company "Csaba Nagy")
 		(comment 1 "SPDX-License-Identifier: CERN-OHL-S-2.0")
 	)
