File: keyboard.kicad_sch (KiCad schematic)
At the start: 86 parts, among them J3 Conn_01x12_Pin, SW10 SW_SPST, SW11 SW_SPST, SW12 SW_SPST, SW13 SW_SPST, SW14 SW_SPST, SW15 SW_SPST, SW16 SW_SPST, SW17 SW_SPST, SW18 SW_SPST, SW19 SW_SPST, SW20 SW_SPST, SW21 SW_SPST, SW22 SW_SPST, SW23 SW_SPST, SW24 SW_SPST, SW25 SW_SPST, SW26 SW_SPST, SW27 SW_SPST, SW28 SW_SPST, SW29 SW_SPST, SW3 SW_SPST, SW30 SW_SPST, SW31 SW_SPST, SW32 SW_SPST, SW33 SW_SPST, SW34 SW_SPST, SW35 SW_SPST, SW36 SW_SPST, SW37 SW_SPST, SW38 SW_SPST, SW39 SW_SPST, SW4 SW_SPST, SW5 SW_SPST, SW6 SW_SPST, SW7 SW_SPST, SW8 SW_SPST, SW9 SW_SPST, U17 M110

Commit message: Routing
Parts:
- SW10, SW11, SW12, SW13, SW14, SW15, SW16, SW17, SW18, SW19, SW20, SW21, SW22, SW23, SW24, SW25, SW26, SW27, SW28, SW29, SW3, SW30, SW31, SW32, SW33, SW34, SW35, SW36, SW37, SW38, SW39, SW4, SW5, SW6, SW7, SW8, SW9: footprint PCM_Jumper_AKL:Jumper_P30.48mm_D1.2mm -> TestPoint:TestPoint_Loop_D3.80mm_Drill2.8mm
Changed lines of the file:
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@@
 			)
 		)
-		(property "Footprint" "PCM_Jumper_AKL:Jumper_P30.48mm_D1.2mm"
+		(property "Footprint" "TestPoint:TestPoint_Loop_D3.80mm_Drill2.8mm"
 			(at 246.38 109.22 0)
 			(effects
@@
 			)
 		)
-		(property "Footprint" "PCM_Jumper_AKL:Jumper_P30.48mm_D1.2mm"
+		(property "Footprint" "TestPoint:TestPoint_Loop_D3.80mm_Drill2.8mm"
 			(at 233.68 71.12 0)
 			(effects
@@
 			)
 		)
-		(property "Footprint" "PCM_Jumper_AKL:Jumper_P30.48mm_D1.2mm"
+		(property "Footprint" "TestPoint:TestPoint_Loop_D3.80mm_Drill2.8mm"
 			(at 220.98 109.22 0)
 			(effects
@@
 			)
 		)
-		(property "Footprint" "PCM_Jumper_AKL:Jumper_P30.48mm_D1.2mm"
+		(property "Footprint" "TestPoint:TestPoint_Loop_D3.80mm_Drill2.8mm"
 			(at 259.08 71.12 0)
 			(effects
@@
 			)
 		)
-		(property "Footprint" "PCM_Jumper_AKL:Jumper_P30.48mm_D1.2mm"
+		(property "Footprint" "TestPoint:TestPoint_Loop_D3.80mm_Drill2.8mm"
 			(at 259.08 109.22 0)
 			(effects
@@
 			)
 		)
-		(property "Footprint" "PCM_Jumper_AKL:Jumper_P30.48mm_D1.2mm"
+		(property "Footprint" "TestPoint:TestPoint_Loop_D3.80mm_Drill2.8mm"
 			(at 195.58 109.22 0)
 			(effects
@@
 			)
 		)
-		(property "Footprint" "PCM_Jumper_AKL:Jumper_P30.48mm_D1.2mm"
+		(property "Footprint" "TestPoint:TestPoint_Loop_D3.80mm_Drill2.8mm"
 			(at 170.18 109.22 0)
 			(effects
@@
 			)
 		)
-		(property "Footprint" "PCM_Jumper_AKL:Jumper_P30.48mm_D1.2mm"
+		(property "Footprint" "TestPoint:TestPoint_Loop_D3.80mm_Drill2.8mm"
 			(at 271.78 33.02 0)
 			(effects
@@
 			)
 		)
-		(property "Footprint" "PCM_Jumper_AKL:Jumper_P30.48mm_D1.2mm"
+		(property "Footprint" "TestPoint:TestPoint_Loop_D3.80mm_Drill2.8mm"
 			(at 233.68 109.22 0)
 			(effects
@@
 			)
 		)
-		(property "Footprint" "PCM_Jumper_AKL:Jumper_P30.48mm_D1.2mm"
+		(property "Footprint" "TestPoint:TestPoint_Loop_D3.80mm_Drill2.8mm"
 			(at 271.78 147.32 0)
 			(effects
@@
 			)
 		)
-		(property "Footprint" "PCM_Jumper_AKL:Jumper_P30.48mm_D1.2mm"
+		(property "Footprint" "TestPoint:TestPoint_Loop_D3.80mm_Drill2.8mm"
 			(at 182.88 109.22 0)
 			(effects
@@
 			)
 		)
-		(property "Footprint" "PCM_Jumper_AKL:Jumper_P30.48mm_D1.2mm"
+		(property "Footprint" "TestPoint:TestPoint_Loop_D3.80mm_Drill2.8mm"
 			(at 144.78 33.02 0)
 			(effects
@@
 			)
 		)
-		(property "Footprint" "PCM_Jumper_AKL:Jumper_P30.48mm_D1.2mm"
+		(property "Footprint" "TestPoint:TestPoint_Loop_D3.80mm_Drill2.8mm"
 			(at 259.08 33.02 0)
 			(effects
@@
 			)
 		)
-		(property "Footprint" "PCM_Jumper_AKL:Jumper_P30.48mm_D1.2mm"
+		(property "Footprint" "TestPoint:TestPoint_Loop_D3.80mm_Drill2.8mm"
 			(at 195.58 33.02 0)
 			(effects
@@
 			)
 		)
-		(property "Footprint" "PCM_Jumper_AKL:Jumper_P30.48mm_D1.2mm"
+		(property "Footprint" "TestPoint:TestPoint_Loop_D3.80mm_Drill2.8mm"
 			(at 246.38 33.02 0)
 			(effects
@@
 			)
 		)
-		(property "Footprint" "PCM_Jumper_AKL:Jumper_P30.48mm_D1.2mm"
+		(property "Footprint" "TestPoint:TestPoint_Loop_D3.80mm_Drill2.8mm"
 			(at 132.08 71.12 0)
 			(effects
@@
 			)
 		)
-		(property "Footprint" "PCM_Jumper_AKL:Jumper_P30.48mm_D1.2mm"
+		(property "Footprint" "TestPoint:TestPoint_Loop_D3.80mm_Drill2.8mm"
 			(at 182.88 33.02 0)
 			(effects
@@
 			)
 		)
-		(property "Footprint" "PCM_Jumper_AKL:Jumper_P30.48mm_D1.2mm"
+		(property "Footprint" "TestPoint:TestPoint_Loop_D3.80mm_Drill2.8mm"
 			(at 208.28 109.22 0)
 			(effects
@@
 			)
 		)
-		(property "Footprint" "PCM_Jumper_AKL:Jumper_P30.48mm_D1.2mm"
+		(property "Footprint" "TestPoint:TestPoint_Loop_D3.80mm_Drill2.8mm"
 			(at 170.18 33.02 0)
 			(effects
@@
 			)
 		)
-		(property "Footprint" "PCM_Jumper_AKL:Jumper_P30.48mm_D1.2mm"
+		(property "Footprint" "TestPoint:TestPoint_Loop_D3.80mm_Drill2.8mm"
 			(at 157.48 109.22 0)
 			(effects
@@
 			)
 		)
-		(property "Footprint" "PCM_Jumper_AKL:Jumper_P30.48mm_D1.2mm"
+		(property "Footprint" "TestPoint:TestPoint_Loop_D3.80mm_Drill2.8mm"
 			(at 208.28 71.12 0)
 			(effects
@@
 			)
 		)
-		(property "Footprint" "PCM_Jumper_AKL:Jumper_P30.48mm_D1.2mm"
+		(property "Footprint" "TestPoint:TestPoint_Loop_D3.80mm_Drill2.8mm"
 			(at 271.78 109.22 0)
 			(effects
@@
 			)
 		)
-		(property "Footprint" "PCM_Jumper_AKL:Jumper_P30.48mm_D1.2mm"
+		(property "Footprint" "TestPoint:TestPoint_Loop_D3.80mm_Drill2.8mm"
 			(at 208.28 33.02 0)
 			(effects
@@
 			)
 		)
-		(property "Footprint" "PCM_Jumper_AKL:Jumper_P30.48mm_D1.2mm"
+		(property "Footprint" "TestPoint:TestPoint_Loop_D3.80mm_Drill2.8mm"
 			(at 157.48 33.02 0)
 			(effects
@@
 			)
 		)
-		(property "Footprint" "PCM_Jumper_AKL:Jumper_P30.48mm_D1.2mm"
+		(property "Footprint" "TestPoint:TestPoint_Loop_D3.80mm_Drill2.8mm"
 			(at 132.08 109.22 0)
 			(effects
@@
 			)
 		)
-		(property "Footprint" "PCM_Jumper_AKL:Jumper_P30.48mm_D1.2mm"
+		(property "Footprint" "TestPoint:TestPoint_Loop_D3.80mm_Drill2.8mm"
 			(at 144.78 71.12 0)
 			(effects
@@
 			)
 		)
-		(property "Footprint" "PCM_Jumper_AKL:Jumper_P30.48mm_D1.2mm"
+		(property "Footprint" "TestPoint:TestPoint_Loop_D3.80mm_Drill2.8mm"
 			(at 132.08 33.02 0)
 			(effects
@@
 			)
 		)
-		(property "Footprint" "PCM_Jumper_AKL:Jumper_P30.48mm_D1.2mm"
+		(property "Footprint" "TestPoint:TestPoint_Loop_D3.80mm_Drill2.8mm"
 			(at 170.18 71.12 0)
 			(effects
@@
 			)
 		)
-		(property "Footprint" "PCM_Jumper_AKL:Jumper_P30.48mm_D1.2mm"
+		(property "Footprint" "TestPoint:TestPoint_Loop_D3.80mm_Drill2.8mm"
 			(at 246.38 71.12 0)
 			(effects
@@
 			)
 		)
-		(property "Footprint" "PCM_Jumper_AKL:Jumper_P30.48mm_D1.2mm"
+		(property "Footprint" "TestPoint:TestPoint_Loop_D3.80mm_Drill2.8mm"
 			(at 195.58 71.12 0)
 			(effects
@@
 			)
 		)
-		(property "Footprint" "PCM_Jumper_AKL:Jumper_P30.48mm_D1.2mm"
+		(property "Footprint" "TestPoint:TestPoint_Loop_D3.80mm_Drill2.8mm"
 			(at 220.98 33.02 0)
 			(effects
@@
 			)
 		)
-		(property "Footprint" "PCM_Jumper_AKL:Jumper_P30.48mm_D1.2mm"
+		(property "Footprint" "TestPoint:TestPoint_Loop_D3.80mm_Drill2.8mm"
 			(at 157.48 71.12 0)
 			(effects
@@
 			)
 		)
-		(property "Footprint" "PCM_Jumper_AKL:Jumper_P30.48mm_D1.2mm"
+		(property "Footprint" "TestPoint:TestPoint_Loop_D3.80mm_Drill2.8mm"
 			(at 233.68 33.02 0)
 			(effects
@@
 			)
 		)
-		(property "Footprint" "PCM_Jumper_AKL:Jumper_P30.48mm_D1.2mm"
+		(property "Footprint" "TestPoint:TestPoint_Loop_D3.80mm_Drill2.8mm"
 			(at 182.88 71.12 0)
 			(effects
@@
 			)
 		)
-		(property "Footprint" "PCM_Jumper_AKL:Jumper_P30.48mm_D1.2mm"
+		(property "Footprint" "TestPoint:TestPoint_Loop_D3.80mm_Drill2.8mm"
 			(at 271.78 71.12 0)
 			(effects
@@
 			)
 		)
-		(property "Footprint" "PCM_Jumper_AKL:Jumper_P30.48mm_D1.2mm"
+		(property "Footprint" "TestPoint:TestPoint_Loop_D3.80mm_Drill2.8mm"
 			(at 144.78 109.22 0)
 			(effects
@@
 			)
 		)
-		(property "Footprint" "PCM_Jumper_AKL:Jumper_P30.48mm_D1.2mm"
+		(property "Footprint" "TestPoint:TestPoint_Loop_D3.80mm_Drill2.8mm"
 			(at 220.98 71.12 0)
 			(effects

Commit message: Start keyboard routing - WIP
Parts:
- D11, D12, D13, D14, D15, D16, D17, D18, D19, D20, D21, D22, D23, D24, D25, D26, D27, D28, D29, D30, D31, D32, D33, D34, D35, D36, D37, D38, D39, D40, D41, D42, D43, D44, D45, D46, D47: footprint Diode_THT:D_DO-35_SOD27_P7.62mm_Horizontal -> Diode_THT:D_DO-35_SOD27_P12.70mm_Horizontal
Changed lines of the file:
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@@
 			)
 		)
-		(property "Footprint" "Diode_THT:D_DO-35_SOD27_P7.62mm_Horizontal"
+		(property "Footprint" "Diode_THT:D_DO-35_SOD27_P12.70mm_Horizontal"
 			(at 157.48 81.28 0)
 			(effects
@@
 			)
 		)
-		(property "Footprint" "Diode_THT:D_DO-35_SOD27_P7.62mm_Horizontal"
+		(property "Footprint" "Diode_THT:D_DO-35_SOD27_P12.70mm_Horizontal"
 			(at 208.28 81.28 0)
 			(effects
@@
 			)
 		)
-		(property "Footprint" "Diode_THT:D_DO-35_SOD27_P7.62mm_Horizontal"
+		(property "Footprint" "Diode_THT:D_DO-35_SOD27_P12.70mm_Horizontal"
 			(at 233.68 81.28 0)
 			(effects
@@
 			)
 		)
-		(property "Footprint" "Diode_THT:D_DO-35_SOD27_P7.62mm_Horizontal"
+		(property "Footprint" "Diode_THT:D_DO-35_SOD27_P12.70mm_Horizontal"
 			(at 271.78 157.48 0)
 			(effects
@@
 			)
 		)
-		(property "Footprint" "Diode_THT:D_DO-35_SOD27_P7.62mm_Horizontal"
+		(property "Footprint" "Diode_THT:D_DO-35_SOD27_P12.70mm_Horizontal"
 			(at 157.48 119.38 0)
 			(effects
@@
 			)
 		)
-		(property "Footprint" "Diode_THT:D_DO-35_SOD27_P7.62mm_Horizontal"
+		(property "Footprint" "Diode_THT:D_DO-35_SOD27_P12.70mm_Horizontal"
 			(at 220.98 43.18 0)
 			(effects
@@
 			)
 		)
-		(property "Footprint" "Diode_THT:D_DO-35_SOD27_P7.62mm_Horizontal"
+		(property "Footprint" "Diode_THT:D_DO-35_SOD27_P12.70mm_Horizontal"
 			(at 246.38 119.38 0)
 			(effects
@@
 			)
 		)
-		(property "Footprint" "Diode_THT:D_DO-35_SOD27_P7.62mm_Horizontal"
+		(property "Footprint" "Diode_THT:D_DO-35_SOD27_P12.70mm_Horizontal"
 			(at 246.38 81.28 0)
 			(effects
@@
 			)
 		)
-		(property "Footprint" "Diode_THT:D_DO-35_SOD27_P7.62mm_Horizontal"
+		(property "Footprint" "Diode_THT:D_DO-35_SOD27_P12.70mm_Horizontal"
 			(at 144.78 43.18 0)
 			(effects
@@
 			)
 		)
-		(property "Footprint" "Diode_THT:D_DO-35_SOD27_P7.62mm_Horizontal"
+		(property "Footprint" "Diode_THT:D_DO-35_SOD27_P12.70mm_Horizontal"
 			(at 195.58 119.38 0)
 			(effects
@@
 			)
 		)
-		(property "Footprint" "Diode_THT:D_DO-35_SOD27_P7.62mm_Horizontal"
+		(property "Footprint" "Diode_THT:D_DO-35_SOD27_P12.70mm_Horizontal"
 			(at 271.78 43.18 0)
 			(effects
@@
 			)
 		)
-		(property "Footprint" "Diode_THT:D_DO-35_SOD27_P7.62mm_Horizontal"
+		(property "Footprint" "Diode_THT:D_DO-35_SOD27_P12.70mm_Horizontal"
 			(at 132.08 119.38 0)
 			(effects
@@
 			)
 		)
-		(property "Footprint" "Diode_THT:D_DO-35_SOD27_P7.62mm_Horizontal"
+		(property "Footprint" "Diode_THT:D_DO-35_SOD27_P12.70mm_Horizontal"
 			(at 132.08 81.28 0)
 			(effects
@@
 			)
 		)
-		(property "Footprint" "Diode_THT:D_DO-35_SOD27_P7.62mm_Horizontal"
+		(property "Footprint" "Diode_THT:D_DO-35_SOD27_P12.70mm_Horizontal"
 			(at 182.88 81.28 0)
 			(effects
@@
 			)
 		)
-		(property "Footprint" "Diode_THT:D_DO-35_SOD27_P7.62mm_Horizontal"
+		(property "Footprint" "Diode_THT:D_DO-35_SOD27_P12.70mm_Horizontal"
 			(at 233.68 43.18 0)
 			(effects
@@
 			)
 		)
-		(property "Footprint" "Diode_THT:D_DO-35_SOD27_P7.62mm_Horizontal"
+		(property "Footprint" "Diode_THT:D_DO-35_SOD27_P12.70mm_Horizontal"
 			(at 220.98 81.28 0)
 			(effects
@@
 			)
 		)
-		(property "Footprint" "Diode_THT:D_DO-35_SOD27_P7.62mm_Horizontal"
+		(property "Footprint" "Diode_THT:D_DO-35_SOD27_P12.70mm_Horizontal"
 			(at 170.18 81.28 0)
 			(effects
@@
 			)
 		)
-		(property "Footprint" "Diode_THT:D_DO-35_SOD27_P7.62mm_Horizontal"
+		(property "Footprint" "Diode_THT:D_DO-35_SOD27_P12.70mm_Horizontal"
 			(at 259.08 119.38 0)
 			(effects
@@
 			)
 		)
-		(property "Footprint" "Diode_THT:D_DO-35_SOD27_P7.62mm_Horizontal"
+		(property "Footprint" "Diode_THT:D_DO-35_SOD27_P12.70mm_Horizontal"
 			(at 182.88 43.18 0)
 			(effects
@@
 			)
 		)
-		(property "Footprint" "Diode_THT:D_DO-35_SOD27_P7.62mm_Horizontal"
+		(property "Footprint" "Diode_THT:D_DO-35_SOD27_P12.70mm_Horizontal"
 			(at 208.28 119.38 0)
 			(effects
@@
 			)
 		)
-		(property "Footprint" "Diode_THT:D_DO-35_SOD27_P7.62mm_Horizontal"
+		(property "Footprint" "Diode_THT:D_DO-35_SOD27_P12.70mm_Horizontal"
 			(at 259.08 43.18 0)
 			(effects
@@
 			)
 		)
-		(property "Footprint" "Diode_THT:D_DO-35_SOD27_P7.62mm_Horizontal"
+		(property "Footprint" "Diode_THT:D_DO-35_SOD27_P12.70mm_Horizontal"
 			(at 170.18 43.18 0)
 			(effects
@@
 			)
 		)
-		(property "Footprint" "Diode_THT:D_DO-35_SOD27_P7.62mm_Horizontal"
+		(property "Footprint" "Diode_THT:D_DO-35_SOD27_P12.70mm_Horizontal"
 			(at 208.28 43.18 0)
 			(effects
@@
 			)
 		)
-		(property "Footprint" "Diode_THT:D_DO-35_SOD27_P7.62mm_Horizontal"
+		(property "Footprint" "Diode_THT:D_DO-35_SOD27_P12.70mm_Horizontal"
 			(at 195.58 81.28 0)
 			(effects
@@
 			)
 		)
-		(property "Footprint" "Diode_THT:D_DO-35_SOD27_P7.62mm_Horizontal"
+		(property "Footprint" "Diode_THT:D_DO-35_SOD27_P12.70mm_Horizontal"
 			(at 271.78 119.38 0)
 			(effects
@@
 			)
 		)
-		(property "Footprint" "Diode_THT:D_DO-35_SOD27_P7.62mm_Horizontal"
+		(property "Footprint" "Diode_THT:D_DO-35_SOD27_P12.70mm_Horizontal"
 			(at 132.08 43.18 0)
 			(effects
@@
 			)
 		)
-		(property "Footprint" "Diode_THT:D_DO-35_SOD27_P7.62mm_Horizontal"
+		(property "Footprint" "Diode_THT:D_DO-35_SOD27_P12.70mm_Horizontal"
 			(at 220.98 119.38 0)
 			(effects
@@
 			)
 		)
-		(property "Footprint" "Diode_THT:D_DO-35_SOD27_P7.62mm_Horizontal"
+		(property "Footprint" "Diode_THT:D_DO-35_SOD27_P12.70mm_Horizontal"
 			(at 182.88 119.38 0)
 			(effects
@@
 			)
 		)
-		(property "Footprint" "Diode_THT:D_DO-35_SOD27_P7.62mm_Horizontal"
+		(property "Footprint" "Diode_THT:D_DO-35_SOD27_P12.70mm_Horizontal"
 			(at 259.08 81.28 0)
 			(effects
@@
 			)
 		)
-		(property "Footprint" "Diode_THT:D_DO-35_SOD27_P7.62mm_Horizontal"
+		(property "Footprint" "Diode_THT:D_DO-35_SOD27_P12.70mm_Horizontal"
 			(at 233.68 119.38 0)
 			(effects
@@
 			)
 		)
-		(property "Footprint" "Diode_THT:D_DO-35_SOD27_P7.62mm_Horizontal"
+		(property "Footprint" "Diode_THT:D_DO-35_SOD27_P12.70mm_Horizontal"
 			(at 246.38 43.18 0)
 			(effects
@@
 			)
 		)
-		(property "Footprint" "Diode_THT:D_DO-35_SOD27_P7.62mm_Horizontal"
+		(property "Footprint" "Diode_THT:D_DO-35_SOD27_P12.70mm_Horizontal"
 			(at 144.78 119.38 0)
 			(effects
@@
 			)
 		)
-		(property "Footprint" "Diode_THT:D_DO-35_SOD27_P7.62mm_Horizontal"
+		(property "Footprint" "Diode_THT:D_DO-35_SOD27_P12.70mm_Horizontal"
 			(at 170.18 119.38 0)
 			(effects
@@
 			)
 		)
-		(property "Footprint" "Diode_THT:D_DO-35_SOD27_P7.62mm_Horizontal"
+		(property "Footprint" "Diode_THT:D_DO-35_SOD27_P12.70mm_Horizontal"
 			(at 271.78 81.28 0)
 			(effects
@@
 			)
 		)
-		(property "Footprint" "Diode_THT:D_DO-35_SOD27_P7.62mm_Horizontal"
+		(property "Footprint" "Diode_THT:D_DO-35_SOD27_P12.70mm_Horizontal"
 			(at 144.78 81.28 0)
 			(effects
@@
 			)
 		)
-		(property "Footprint" "Diode_THT:D_DO-35_SOD27_P7.62mm_Horizontal"
+		(property "Footprint" "Diode_THT:D_DO-35_SOD27_P12.70mm_Horizontal"
 			(at 195.58 43.18 0)
 			(effects
@@
 			)
 		)
-		(property "Footprint" "Diode_THT:D_DO-35_SOD27_P7.62mm_Horizontal"
+		(property "Footprint" "Diode_THT:D_DO-35_SOD27_P12.70mm_Horizontal"
 			(at 157.48 43.18 0)
 			(effects
