File: vca_envelope.kicad_sch (KiCad schematic)
At the start: 20 parts, among them J9 Conn_01x06_Pin, Q3 BC237, U11 4001, U12 4066, U13 Opamp_Dual

Commit message: Routing
Connections:
- net GND: now also R30.2; no longer RV12.2
- net at R30.1: now also RV12.2; no longer U12.4
- net at RV12.1: now also U12.4; no longer R30.2
Other:
- moved on the sheet: R30, RV12
Changed lines of the file:
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@@
 	(text "RELEASE"
 		(exclude_from_sim no)
-		(at 177.038 135.89 0)
+		(at 165.862 133.35 0)
 		(effects
 			(font
@@
 	)
 	(no_connect
-		(at 171.45 144.78)
+		(at 171.45 132.08)
 	)
 	(no_connect
@@
 	(wire
 		(pts
-			(xy 171.45 132.08) (xy 171.45 137.16)
-		)
-		(stroke
-			(width 0)
-			(type default)
-		)
-	)
-	(wire
-		(pts
 			(xy 171.45 99.06) (xy 171.45 102.87)
 		)
@@
 	(wire
 		(pts
+			(xy 176.53 132.08) (xy 176.53 128.27)
+		)
+		(stroke
+			(width 0)
+			(type default)
+		)
+	)
+	(wire
+		(pts
 			(xy 148.59 58.42) (xy 162.56 58.42)
 		)
@@
 	(wire
 		(pts
-			(xy 176.53 140.97) (xy 175.26 140.97)
+			(xy 176.53 128.27) (xy 175.26 128.27)
 		)
 		(stroke
@@
 	(wire
 		(pts
-			(xy 176.53 144.78) (xy 176.53 140.97)
+			(xy 176.53 144.78) (xy 176.53 139.7)
 		)
 		(stroke
@@
 	(symbol
 		(lib_id "Device:R")
-		(at 171.45 128.27 0)
+		(at 176.53 135.89 0)
 		(unit 1)
 		(exclude_from_sim no)
@@
 		(fields_autoplaced yes)
 		(property "Reference" "R30"
-			(at 173.99 126.9999 0)
+			(at 179.07 134.6199 0)
 			(effects
 				(font
@@
 		)
 		(property "Value" "1K"
-			(at 173.99 129.5399 0)
+			(at 179.07 137.1599 0)
 			(effects
 				(font
@@
 		)
 		(property "Footprint" "Resistor_THT:R_Axial_DIN0207_L6.3mm_D2.5mm_P15.24mm_Horizontal"
-			(at 169.672 128.27 90)
+			(at 174.752 135.89 90)
 			(effects
 				(font
@@
 		)
 		(property "Datasheet" "~"
-			(at 171.45 128.27 0)
+			(at 176.53 135.89 0)
 			(effects
 				(font
@@
 		)
 		(property "Description" "Resistor"
-			(at 171.45 128.27 0)
+			(at 176.53 135.89 0)
 			(effects
 				(font
@@
 	(symbol
 		(lib_id "Device:R_Potentiometer")
-		(at 171.45 140.97 0)
+		(at 171.45 128.27 0)
 		(unit 1)
 		(exclude_from_sim no)
@@
 		(on_board yes)
 		(dnp no)
+		(fields_autoplaced yes)
 		(property "Reference" "RV12"
-			(at 168.91 139.6999 0)
+			(at 168.91 126.9999 0)
 			(effects
 				(font
@@
 		)
 		(property "Value" "2M2B"
-			(at 168.91 142.2399 0)
+			(at 168.91 129.5399 0)
 			(effects
 				(font
@@
 		)
 		(property "Footprint" "Potentiometer_THT:Potentiometer_Omeg_PC16BU_Vertical"
-			(at 171.45 140.97 0)
+			(at 171.45 128.27 0)
 			(effects
 				(font
@@
 		)
 		(property "Datasheet" "~"
-			(at 171.45 140.97 0)
+			(at 171.45 128.27 0)
 			(effects
 				(font
@@
 		)
 		(property "Description" "Potentiometer"
-			(at 171.45 140.97 0)
-			(effects
-				(font
+			(at 171.45 128.27 0)
+			(effects
+				(font

Commit message: Start keyboard routing - WIP
Parts:
- C18: footprint Capacitor_THT:C_Disc_D5.0mm_W2.5mm_P5.00mm -> Capacitor_THT:C_Rect_L11.0mm_W2.8mm_P10.00mm_MKT
Changed lines of the file:
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@@
 			)
 		)
-		(property "Footprint" "Capacitor_THT:C_Disc_D5.0mm_W2.5mm_P5.00mm"
+		(property "Footprint" "Capacitor_THT:C_Rect_L11.0mm_W2.8mm_P10.00mm_MKT"
 			(at 190.8048 101.6 0)
 			(effects

Commit message: Update README, add license to sheets
Other:
- title: (none) -> JEN SX-1000
Changed lines of the file:
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@@
 	(generator_version "9.0")
 	(paper "A4")
+	(title_block
+		(title "JEN SX-1000")
+		(comment 1 "SPDX-License-Identifier: CERN-OHL-S-2.0")
+	)
 	(text "DECAY"
 		(exclude_from_sim no)
