File: vca_envelope.kicad_sch (KiCad schematic)
At the start: 20 parts, among them J9 Conn_01x06_Pin, Q3 BC237, U11 4001, U12 4066, U13 Opamp_Dual

Commit message: Update sheets
Other:
- company: (none) -> Csaba Nagy
Changed lines of the file:
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@@
 	(title_block
 		(title "JEN SX-1000")
+		(company "Csaba Nagy")
 		(comment 1 "SPDX-License-Identifier: CERN-OHL-S-2.0")
 	)
