File: noise.kicad_sch (KiCad schematic)
At the start: 26 parts, among them J2 Conn_01x04_Pin, SW1 SW_SP3T, U20 LF351N, U5 MM5837

Commit message: Update README, add license to sheets
Other:
- title: (none) -> JEN SX-1000
Changed lines of the file:
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@@
 	(generator_version "9.0")
 	(paper "A4")
+	(title_block
+		(title "JEN SX-1000")
+		(comment 1 "SPDX-License-Identifier: CERN-OHL-S-2.0")
+	)
 	(rectangle
 		(start 72.39 121.92)

Commit message: Update sheets
Other:
- company: (none) -> Csaba Nagy
Changed lines of the file:
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@@
 	(title_block
 		(title "JEN SX-1000")
+		(company "Csaba Nagy")
 		(comment 1 "SPDX-License-Identifier: CERN-OHL-S-2.0")
 	)
