File: vca.kicad_sch (KiCad schematic)
At the start: 15 parts, among them J5 Conn_01x09_Pin, Q1 BC309C, U6 CA3080, U7 LM741

Commit message: Routing
Connections:
- net +12V: now also RT4.3; no longer RT4.1
- net -12V: now also RT4.1; no longer RT4.3
- net GND: now also RV3.1; no longer RV3.3
- net at R16.2, U7.6: now also RV3.3; no longer RV3.1
Changed lines of the file:
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@@
+	(wire
+		(pts
+			(xy 26.67 17.78) (xy 31.75 17.78)
+		)
+		(stroke
+			(width 0)
+			(type default)
+		)
+	)
 	(wire
 		(pts
@@
 		)
 	)
+	(hierarchical_label "+15V"
+		(shape input)
+		(at 26.67 17.78 180)
+		(effects
+			(font
+				(size 1.27 1.27)
+			)
+			(justify right)
+		)
+	)
 	(hierarchical_label "+12V"
 		(shape input)
@@
 		(lib_id "Device:R_Potentiometer")
 		(at 191.77 134.62 0)
+		(mirror x)
 		(unit 1)
 		(exclude_from_sim no)
@@
 		(dnp no)
 		(property "Reference" "RV3"
-			(at 189.23 133.3499 0)
+			(at 189.23 132.0799 0)
 			(effects
 				(font
@@
 		)
 		(property "Value" "10KA"
-			(at 189.23 135.8899 0)
+			(at 189.23 134.6199 0)
 			(effects
 				(font
@@
 		)
 		(property "Description" "OUTPUT VOLUME"
-			(at 200.66 139.7 0)
-			(effects
-				(font
-					(size 1.27 1.27)
-				)
+			(at 188.722 140.716 0)
+			(effects
+				(font
+					(size 1.27 1.27)
+				)
+				(justify right)
 			)
 		)
@@
 				(path "/3c53febc-5769-4c45-8f8f-0aba2c04e944/75668585-e3c2-431b-bb9e-906e88891a90"
 					(reference "#PWR029")
+					(unit 1)
+				)
+			)
+		)
+	)
+	(symbol
+		(lib_id "power:+15V")
+		(at 31.75 17.78 0)
+		(unit 1)
+		(exclude_from_sim no)
+		(in_bom yes)
+		(on_board yes)
+		(dnp no)
+		(fields_autoplaced yes)
+		(property "Reference" "#PWR0168"
+			(at 31.75 21.59 0)
+			(effects
+				(font
+					(size 1.27 1.27)
+				)
+				(hide yes)
+			)
+		)
+		(property "Value" "+15V"
+			(at 31.75 12.7 0)
+			(effects
+				(font
+					(size 1.27 1.27)
+				)
+			)
+		)
+		(property "Footprint" ""
+			(at 31.75 17.78 0)
+			(effects
+				(font
+					(size 1.27 1.27)
+				)
+				(hide yes)
+			)
+		)
+		(property "Datasheet" ""
+			(at 31.75 17.78 0)
+			(effects
+				(font
+					(size 1.27 1.27)
+				)
+				(hide yes)
+			)
+		)
+		(property "Description" "Power symbol creates a global label with name \"+15V\""
+			(at 31.75 17.78 0)
+			(effects
+				(font
+					(size 1.27 1.27)
+				)
+				(hide yes)
+			)
+		)
+		(pin "1"
+		)
+		(instances
+			(project "jensx1000"
+				(path "/3c53febc-5769-4c45-8f8f-0aba2c04e944/75668585-e3c2-431b-bb9e-906e88891a90"
+					(reference "#PWR0168")
 					(unit 1)
 				)
@@
 		(lib_id "Device:R_Potentiometer_Trim")
 		(at 111.76 92.71 0)
-		(unit 1)
-		(exclude_from_sim no)
-		(in_bom yes)
-		(on_board yes)
-		(dnp no)
+		(mirror x)
+		(unit 1)
+		(exclude_from_sim no)
+		(in_bom yes)
+		(on_board yes)
+		(dnp no)
+		(fields_autoplaced yes)
 		(property "Reference" "RT4"
-			(at 109.22 91.4399 0)
+			(at 109.22 90.1699 0)
 			(effects
 				(font
@@
 		)
 		(property "Value" "100R"
-			(at 109.22 93.9799 0)
+			(at 109.22 92.7099 0)
 			(effects
 				(font
@@
 		)
 		(property "Description" "VCA OFFSET"
-			(at 118.618 97.028 0)
-			(effects
-				(font
-					(size 1.27 1.27)
-				)
-			)
-		)
+			(at 109.22 95.2499 0)
+			(effects
+				(font
+					(size 1.27 1.27)
+				)
+				(justify right)
+			)
+		)

Commit message: Update README, add license to sheets
Other:
- title: (none) -> JEN SX-1000
Changed lines of the file:
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@@
 	(generator_version "9.0")
 	(paper "A4")
+	(title_block
+		(title "JEN SX-1000")
+		(comment 1 "SPDX-License-Identifier: CERN-OHL-S-2.0")
+	)
 	(text "VOLUME"
 		(exclude_from_sim no)

Commit message: Update sheets
Other:
- company: (none) -> Csaba Nagy
Changed lines of the file:
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@@
 	(title_block
 		(title "JEN SX-1000")
+		(company "Csaba Nagy")
 		(comment 1 "SPDX-License-Identifier: CERN-OHL-S-2.0")
 	)
