File: vcf.kicad_sch (KiCad schematic)
At the start: 51 parts, among them J6 Conn_01x11_Pin, Q4 BC307, U19 Opamp_Dual, U24 LM13700, U25 LM13700

Commit message: Start keyboard routing - WIP
Parts:
- C8: footprint Capacitor_THT:CP_Radial_D8.0mm_P3.80mm -> Capacitor_THT:CP_Radial_D10.0mm_P7.50mm
Changed lines of the file:
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@@
 			)
 		)
-		(property "Footprint" "Capacitor_THT:CP_Radial_D8.0mm_P3.80mm"
+		(property "Footprint" "Capacitor_THT:CP_Radial_D10.0mm_P7.50mm"
 			(at 31.4452 147.32 0)
 			(effects

Commit message: Update README, add license to sheets
Other:
- title: (none) -> JEN SX-1000
Changed lines of the file:
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@@
 	(generator_version "9.0")
 	(paper "A4")
+	(title_block
+		(title "JEN SX-1000")
+		(comment 1 "SPDX-License-Identifier: CERN-OHL-S-2.0")
+	)
 	(rectangle
 		(start 13.97 128.27)

Commit message: Update sheets
Other:
- company: (none) -> Csaba Nagy
Changed lines of the file:
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@@
 	(title_block
 		(title "JEN SX-1000")
+		(company "Csaba Nagy")
 		(comment 1 "SPDX-License-Identifier: CERN-OHL-S-2.0")
 	)
