File: vcf_envelope.kicad_sch (KiCad schematic)
At the start: 19 parts, among them Q2 BC237, U15 4066, U8 4001, U9 Opamp_Dual

Commit message: Start keyboard routing - WIP
Parts:
- R18: footprint Resistor_THT:R_Axial_DIN0207_L6.3mm_D2.5mm_P15.24mm_Horizontal -> Resistor_THT:R_Axial_DIN0309_L9.0mm_D3.2mm_P12.70mm_Horizontal
Changed lines of the file:
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@@
 			)
 		)
-		(property "Footprint" "Resistor_THT:R_Axial_DIN0207_L6.3mm_D2.5mm_P15.24mm_Horizontal"
+		(property "Footprint" "Resistor_THT:R_Axial_DIN0309_L9.0mm_D3.2mm_P12.70mm_Horizontal"
 			(at 129.032 44.45 90)
 			(effects

Commit message: Update README, add license to sheets
Other:
- title: (none) -> JEN SX-1000
Changed lines of the file:
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@@
 	(generator_version "9.0")
 	(paper "A4")
+	(title_block
+		(title "JEN SX-1000")
+		(comment 1 "SPDX-License-Identifier: CERN-OHL-S-2.0")
+	)
 	(text "DECAY"
 		(exclude_from_sim no)

Commit message: Update sheets
Other:
- company: (none) -> Csaba Nagy
Changed lines of the file:
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@@
 	(title_block
 		(title "JEN SX-1000")
+		(company "Csaba Nagy")
 		(comment 1 "SPDX-License-Identifier: CERN-OHL-S-2.0")
 	)
